File: PCB/PPMInspect.kicad_pcb (KiCad board)
At the start: 2 copper layers, 60 x 97.5 mm, 15 parts, among them J1 Vcc, J2 LCD I2C, J3 Pwr Switch, J4 Data In, SW1 UP/NEXT, SW2 ENTER, SW3 DOWN/RST

Commit message: Microscope grid fix. KiCad new version. V0.9.18
Other:
- net class Default removed
